File: hw/raspi-zero-hat.sch (KiCad schematic (older format))
At the start: 13 parts, among them J1 Screw_Terminal_01x02, J2 Screw_Terminal_01x03, K1 G5LE-1, P1 Conn_02x20_Odd_Even, Q1 MMBT3904

Commit message: moved relay control pin to pin 10 (pin 8 was pulled up on boot, causing an unintended relay toggle).
Connections:
- wire segments 83 -> 82
Changed lines of the file:
@@
 EESchema Schematic File Version 4
-LIBS:raspi-zero-hat-cache
 EELAYER 26 0
 EELAYER END
@@
 Wire Wire Line
 	7650 2600 6900 2600
-Wire Wire Line
-	2900 1500 4200 1500
 $Comp
 L Device:LED D2
@@
 	5850 2100 5600 2100
 Wire Wire Line
-	5600 2100 5600 1400
-Wire Wire Line
-	5600 1400 2900 1400
+	5600 1500 5600 2100
+Wire Wire Line
+	2900 1500 5600 1500
 $EndSCHEMATC
